Commit message: Add second arm and cylinders, update to new optimizer (icra2016)

File: urdf/cylinder_obstacle.urdf (robot description, URDF)
Before this commit: robot cylinder_obstacle, 1 links, 0 joints
Links:
- added link l_cylinder2; collision cylinder length=0.4 radius=0.2; visual cylinder length=0.4 radius=0.2
- added link l_cylinder3; collision cylinder length=0.4 radius=0.2; visual cylinder length=0.4 radius=0.2
- link obstacle_base: mass 1.0 -> None
Joints:
- added joint j_cylinder2: type fixed, parent obstacle_base, child l_cylinder2, origin xyz=0 0 0
- added joint j_cylinder3: type fixed, parent obstacle_base, child l_cylinder3, origin xyz=0 0 0

File: urdf/object.urdf (robot description, URDF)
Before this commit: robot object, 7 links, 6 joints
Links:
- added link l_object_second_arm_one; collision cylinder length=0.8 radius=0.05; visual cylinder length=0.8 radius=0.05
- added link l_object_second_arm_two; collision cylinder length=0.8 radius=0.05; visual cylinder length=0.8 radius=0.05
- added link l_sphere2_second_arm; collision sphere radius=0.1; visual sphere radius=0.1
- added link l_sphere3_second_arm; collision sphere radius=0.1; visual sphere radius=0.1
Joints:
- added joint j_object_second_arm_one: type revolute, parent l_object_one, child l_object_second_arm_one, origin xyz=0 0 0, axis 0 0 1, limit lower=-3.14 upper=1.7 effort=1 velocity=1
- added joint j_object_second_arm_two: type revolute, parent l_object_second_arm_one, child l_object_second_arm_two, origin xyz=0.8 0 0, axis 0 0 1, limit lower=-2.9 upper=2.9 effort=1 velocity=1
- added joint j_sphere2_second_arm: type fixed, parent l_object_second_arm_one, child l_sphere2_second_arm, origin xyz=0 0 0
- added joint j_sphere3_second_arm: type fixed, parent l_object_second_arm_two, child l_sphere3_second_arm, origin xyz=0 0 0
- joint j_object_two: limit lower=0.1 upper=3 effort=1 velocity=1 -> lower=-2 upper=3 effort=1 velocity=1

Commit message: Comment second cylinder, enhance script

File: urdf/cylinder_obstacle.urdf (robot description, URDF)
Before this commit: robot cylinder_obstacle, 3 links, 2 joints
Links:
- removed link l_cylinder2
- removed link l_cylinder3
Joints:
- removed joint j_cylinder2
- removed joint j_cylinder3
