Commit message: Add collision-checking for the robot spheres

File: urdf/object.urdf (robot description, URDF)
Before this commit: robot object, 7 links, 6 joints
Links:
- link l_sphere2: geometry collision sphere radius=0.1; visual sphere radius=0.1
- link l_sphere3: geometry collision sphere radius=0.1; visual sphere radius=0.1

Commit message: Scripts and URDF/SRDF modifications:
* base-link is now fixed, adapt cylinder color
* still no-collision-checking between consecutive arms because capsules are colliding
* update script to TADR2, add convergence graphs

File: urdf/object.urdf (robot description, URDF)
Before this commit: robot object, 11 links, 10 joints
Links:
- link base_link: geometry collision cylinder length=1 radius=0.02; visual cylinder length=1 radius=0.02
- link l_object_second_arm_one: geometry collision cylinder length=0.72 radius=0.05; visual cylinder length=0.72 radius=0.05
- link l_object_second_arm_two: geometry collision cylinder length=0.72 radius=0.05; visual cylinder length=0.72 radius=0.05
- link l_object_three: geometry collision cylinder length=0.72 radius=0.05; visual cylinder length=0.72 radius=0.05
- link l_object_two: geometry collision cylinder length=0.72 radius=0.05; visual cylinder length=0.72 radius=0.05
Joints:
- joint j_object_one: axis 1 0 0 -> (none); limit lower=-1.5 upper=1.5 effort=1 velocity=1 -> (none); origin xyz=0 0 0 -> xyz=-0.2 0 0; type prismatic -> fixed
- joint j_object_second_arm_one: limit lower=-3.14 upper=1.7 effort=1 velocity=1 -> lower=-3.14159 upper=3.14159 effort=1 velocity=1
- joint j_object_second_arm_two: limit lower=-2.9 upper=2.9 effort=1 velocity=1 -> lower=-3.14159 upper=3.14159 effort=1 velocity=1
- joint j_object_three: limit lower=-2.9 upper=2.9 effort=1 velocity=1 -> lower=-3.14159 upper=3.14159 effort=1 velocity=1
- joint j_object_two: limit lower=-2 upper=3 effort=1 velocity=1 -> lower=-3.14159 upper=3.14159 effort=1 velocity=1
